File: pBITzBackplaneMezzanine/USBPorts.kicad_sch (KiCad schematic)
At the start: 30 parts, among them J1 USB3_A_Stacked, J2 Conn_01x04, J3 Conn_01x04, U1 FE1.1S-BSOP28BCN, U2 MAX3421EETJ_T, U3 CD74HC4050M96, Y1 ABL-12.000MHZ-B2, Y2 ABL-12.000MHZ-B2

Commit message: First pass of validation
Connections:
- net DM1: now also J1.2 (D1-); no longer J1.3 (D1+)
- net DM2: now also J1.11 (D2-); no longer J1.12 (D2+)
- net DP1: now also J1.3 (D1+); no longer J1.2 (D1-)
- net DP2: now also J1.12 (D2+); no longer J1.11 (D2-)
Changed lines of the file:
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@@
 	)
 	(label "DP2"
-		(at 351.79 59.69 0)
+		(at 351.79 62.23 0)
 		(effects
 			(font
@@
 	)
 	(label "DM1"
-		(at 351.79 109.22 0)
+		(at 351.79 106.68 0)
 		(effects
 			(font
@@
 	)
 	(label "DM2"
-		(at 351.79 62.23 0)
+		(at 351.79 59.69 0)
 		(effects
 			(font
@@
 	)
 	(label "DP1"
-		(at 351.79 106.68 0)
-		(effects
-			(font
+		(at 351.79 109.22 0)
+		(effects
+			(font
