File: pBITzBackplaneMezzanine/USBPorts.kicad_sch (KiCad schematic)
At the start: 30 parts, among them J1 USB3_A_Stacked, J2 Conn_01x04, J3 Conn_01x04, U1 FE1.1S-BSOP28BCN, U2 MAX3421EETJ_T, U3 CD74HC4050M96, Y1 ABL-12.000MHZ-B2, Y2 ABL-12.000MHZ-B2

Commit message: Corrections post review
Parts:
- added C16: 1u, Capacitor_SMD:C_0603_1608Metric, symbol Device:C
- added R7: 10k, Resistor_SMD:R_0603_1608Metric, symbol Device:R
Connections:
- net +3V3: now also R7.1
- net GND: now also C16.1
- net ~{USB_INT}: now also R7.2
- net at U2.22 (VBCOMP): now also C16.2
- no-connect marks 34 -> 33
