File: pBITzBackplaneMezzanine/USBPorts.kicad_sch (KiCad schematic)
At the start: 32 parts, among them J1 USB3_A_Stacked, J2 Conn_01x04, J3 Conn_01x04, U1 FE1.1S-BSOP28BCN, U2 MAX3421EETJ_T, U3 CD74HC4050M96, Y1 ABL-12.000MHZ-B2, Y2 ABL-12.000MHZ-B2

Commit message: Fixed the footprint for the FE1.1 (missing file)
Parts:
- U1: footprint Package_SO:SSOP-28_5.3x10.2mm_P0.65mm -> Package_SO:SSOP-28_3.9x9.9mm_P0.635mm
Changed lines of the file:
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@@
 			)
 		)
-		(property "Footprint" "Package_SO:SSOP-28_5.3x10.2mm_P0.65mm"
+		(property "Footprint" "Package_SO:SSOP-28_3.9x9.9mm_P0.635mm"
 			(at 255.27 50.8 0)
 			(hide yes)
