File: pBITzBackplaneMezzanine/pBITzBackplaneMezzanine.kicad_pcb (KiCad board)
At the start: 4 copper layers, 99.9 x 80.4 mm, 41 parts, among them J1 USB3_A_Stacked, J2 Conn_01x04, J3 Conn_01x04, J4 10067847-001RLF, J5 Conn_02x10_Odd_Even, U1 FE1.1S-BSOP28BCN, U2 MAX3421EETJ_T, U3 CD74HC4050M96, U4 CD74HC4050M96, Y1 ABL-12.000MHZ-B2, Y2 ABL-12.000MHZ-B2

Commit message: Corrections post review
Parts:
- added C16: 1u, Capacitor_SMD:C_0603_1608Metric, F.Cu at (453.3, 163.3)
- added R7: 10k, Resistor_SMD:R_0603_1608Metric, F.Cu at (455.7, 165.6)
- moved J4 10.4 mm to (400.0, 211.7)
Connections:
- U2 pad 22: unconnected-(U2-VBCOMP-Pad22) -> Net-(U2-VBCOMP)
- U3 pad 5: /MezzanineConnector/SPI_CS1 -> /MezzanineConnector/SPI_CS0
- U4 pad 11: /MezzanineConnector/SPI_CS0 -> /MezzanineConnector/SPI_CS1
Routing:
- net GND: track 43.6 -> 65.3 mm, vias 27 -> 28
- net /MezzanineConnector/SPI_CS1: track 47.7 -> 65.1 mm
- net +3V3: track 130.2 -> 144.2 mm
- net /SD_Card/CLK: track 19.9 -> 30.4 mm
- net /SD_Card/~{CS}: track 7.01 -> 17.5 mm
- net /SD_Card/MOSI: track 7.06 -> 17.5 mm
- net /MezzanineConnector/~{SD_PRESENT}: track 85.9 -> 96.4 mm
- net /MezzanineConnector/MISO: track 120.9 -> 130.5 mm
- net Net-(U2-VBCOMP): track 0.00 -> 6.52 mm, vias 0 -> 2
- net /MezzanineConnector/SPI_CS0: track 59.3 -> 53.7 mm
- net /MezzanineConnector/~{SPI_INT}: track 23.2 -> 24.3 mm
Other:
- board text added: "DNP"
