File: pBITzBackplaneMezzanine/MezzanineConnector.kicad_sch (KiCad schematic)
At the start: 5 parts, among them J5 Conn_02x10_Odd_Even

Commit message: Corrections post review
Changed lines of the file:
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@@
 	)
 	(symbol
-		(lib_id "power:+5V")
+		(lib_id "power:+3V3")
 		(at 184.15 242.57 0)
-		(mirror y)
 		(unit 1)
 		(body_style 1)
@@
 		(in_pos_files yes)
 		(dnp no)
-		(property "Reference" "#PWR063"
+		(fields_autoplaced yes)
+		(property "Reference" "#PWR037"
 			(at 184.15 246.38 0)
 			(hide yes)
@@
 			)
 		)
-		(property "Description" "Power symbol creates a global label with name \"+5V\""
+		(property "Description" "Power symbol creates a global label with name \"+3V3\""
 			(at 184.15 242.57 0)
 			(hide yes)
@@
 			(project "pBITzBackplaneMezzanine"
 				(path "/d6d8aa35-1d9d-4c27-8a6c-fa24f1b19dce/50888a69-9ed2-4153-90b2-5bf201cc034f"
-					(reference "#PWR063")
+					(reference "#PWR037")
 					(unit 1)
 				)
