File: pBITzBackplaneMezzanine/pBITzBackplaneMezzanine.kicad_sch (KiCad schematic)
At the start: 0 parts

Commit message: Corrections post review
Changed lines of the file:
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@@
 		)
 		(pin "SPI_CS0" output
-			(at 149.86 123.19 90)
+			(at 144.78 123.19 90)
 			(effects
 				(font
@@
 		)
 		(pin "SPI_CS1" output
-			(at 144.78 123.19 90)
+			(at 149.86 123.19 90)
 			(effects
 				(font
