File: pBITzBackplane/pBITzBackplane.kicad_pcb (KiCad board)
At the start: 4 copper layers, 243.8 x 243.8 mm, 55 parts, among them J1 ATX-24, J6 pBITzBus, J7 Conn_02x10_Odd_Even, Q1 BSS138, SW1 SW_Push, U1 ATtiny85-20P

Commit message: Fixed the location of the IDC connector the the mezannine
Parts:
- added REF**: OSHW-Logo2_7.3x6mm_SilkScreen, Symbol:OSHW-Logo2_7.3x6mm_SilkScreen, F.Cu at (245.1, 396.3)
- moved J7 8.05 mm to (258.9, 341.0)
Routing:
- net /Backplane/~{SPI_CS0}: track 369.1 -> 289.0 mm, vias 3 -> 4
- net /Backplane/MOSI: track 368.7 -> 292.3 mm, vias 2 -> 4
- net /Backplane/MISO: track 371.9 -> 295.7 mm, vias 3 -> 4
- net /Backplane/~{SPI_CS1}: track 363.0 -> 289.1 mm, vias 2 -> 4
- net /Backplane/~{SPI_INT}: track 354.3 -> 289.4 mm, vias 3 -> 4
- net +3V3: track 558.3 -> 534.0 mm
- net /Backplane/~{SPI_CD}: track 259.6 -> 259.0 mm
- net /Backplane/SPI_CLK: track 263.6 -> 263.0 mm, vias 8 -> 9
Other:
- copper layers 4 -> 6
