File: pBITzBackplane/pBITzBackplane.kicad_pcb (KiCad board)
At the start: 6 copper layers, 243.8 x 243.8 mm, 56 parts, among them J1 ATX-24, J6 pBITzBus, J7 Conn_02x10_Odd_Even, Q1 BSS138, SW1 SW_Push, U1 ATtiny85-20P

Commit message: updated part #s
Parts:
- removed REF**: OSHW-Logo2_7.3x6mm_SilkScreen, Symbol:OSHW-Logo2_7.3x6mm_SilkScreen
