File: pBITzBackplane/Backplane.kicad_sch (KiCad schematic)
At the start: 20 parts, among them J2 pBITzBus, J3 pBITzBus, J4 pBITzBus, J5 pBITzBus, J6 pBITzBus, J7 Conn_02x10_Odd_Even

Commit message: updated the pullups for the power on sequence pins
Connections:
- net SLK_CLK renamed SPI_CLK
Changed lines of the file:
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@@
 		)
 	)
-	(label "SLK_CLK"
+	(label "SPI_CLK"
 		(at 175.26 57.15 0)
 		(effects
@@
 		)
 	)
-	(label "SLK_CLK"
+	(label "SPI_CLK"
 		(at 478.79 57.15 0)
 		(effects
@@
 		)
 	)
-	(label "SLK_CLK"
+	(label "SPI_CLK"
 		(at 269.24 57.15 0)
 		(effects
@@
 		)
 	)
-	(label "SLK_CLK"
+	(label "SPI_CLK"
 		(at 275.59 227.33 0)
 		(effects
@@
 		)
 	)
-	(label "SLK_CLK"
+	(label "SPI_CLK"
 		(at 372.11 57.15 0)
 		(effects
@@
 		)
 	)
-	(label "SLK_CLK"
+	(label "SPI_CLK"
 		(at 72.39 58.42 0)
 		(effects

Commit message: Changed the pBITz backplane connector from a PCIe 8x to a DIN 41612 connector.
Parts:
- removed J2, J3, J4, J5: pBITzBus, Footprints:AMPHENOL_10018783-10202TLF, symbol pBITz:pBITzBus
- removed RN1, RN2: 4820P-2-472LF, Footprints:SOIC127P762X240-20N, symbol 4820P-2-472LF:4820P-2-472LF
- removed RN3, RN4: 4816P-T02-472LF, Footprints:4816PT02472LF, symbol 4816P-T02-472LF:4816P-T02-472LF
- added J10, J11, J8, J9: (no value), Footprints:AMPHENOL_86093968114T55F1LF, symbol pBITz:pBITzBus_DIN
- added RN10, RN5, RN6, RN7, RN8, RN9: 4614X-101-472LF, Resistor_THT:R_Array_SIP14, symbol Device:R_Network13
Connections:
- net +3V3: now also J10.A3 (+3V3), J10.A4 (+3V3), J10.B3 (+3V3), J10.B4 (+3V3), J11.A3 (+3V3), J11.A4 (+3V3), J11.B3 (+3V3), J11.B4 (+3V3), J8.A3 (+3V3), J8.A4 (+3V3), J8.B3 (+3V3), J8.B4 (+3V3), J9.A3 (+3V3), J9.A4 (+3V3), J9.B3 (+3V3), J9.B4 (+3V3)
- net +5V: now also J10.A1 (+5V), J10.A2 (+5V), J10.B1 (+5V), J10.B2 (+5V), J11.A1 (+5V), J11.A2 (+5V), J11.B1 (+5V), J11.B2 (+5V), J8.A1 (+5V), J8.A2 (+5V), J8.B1 (+5V), J8.B2 (+5V), J9.A1 (+5V), J9.A2 (+5V), J9.B1 (+5V), J9.B2 (+5V), RN10.1 (common), RN5.1 (common), RN6.1 (common), RN7.1 (common), RN8.1 (common), RN9.1 (common)
- net A0: now also J10.A21 (A0), J11.A21 (A0), J8.A21 (A0), J9.A21 (A0), RN8.4 (R3)
- net A1: now also J10.B21 (A1), J11.B21 (A1), J8.B21 (A1), J9.B21 (A1), RN9.4 (R3)
- net A10: now also J10.B24 (A10), J11.B24 (A10), J8.B24 (A10), J9.B24 (A10), RN9.7 (R6)
- net A11: now also J10.C24 (A11), J11.C24 (A11), J8.C24 (A11), J9.C24 (A11), RN10.7 (R6)
- net A12: now also J10.A25 (A12), J11.A25 (A12), J8.A25 (A12), J9.A25 (A12), RN8.8 (R7)
- net A13: now also J10.B25 (A13), J11.B25 (A13), J8.B25 (A13), J9.B25 (A13), RN9.8 (R7)
- net A14: now also J10.C25 (A14), J11.C25 (A14), J8.C25 (A14), J9.C25 (A14), RN10.8 (R7)
- net A15: now also J10.A26 (A15), J11.A26 (A15), J8.A26 (A15), J9.A26 (A15), RN8.9 (R8)
- net A16: now also J10.B26 (A16), J11.B26 (A16), J8.B26 (A16), J9.B26 (A16), RN9.9 (R8)
- net A17: now also J10.C26 (A17), J11.C26 (A17), J8.C26 (A17), J9.C26 (A17), RN10.9 (R8)
- net A18: now also J10.A27 (A18), J11.A27 (A18), J8.A27 (A18), J9.A27 (A18), RN8.10 (R9)
- net A19: now also J10.B27 (A19), J11.B27 (A19), J8.B27 (A19), J9.B27 (A19), RN9.10 (R9)
- net A2: now also J10.C21 (A2), J11.C21 (A2), J8.C21 (A2), J9.C21 (A2), RN10.4 (R3)
- net A20: now also J10.C27 (A20), J11.C27 (A20), J8.C27 (A20), J9.C27 (A20), RN10.10 (R9)
- net A21: now also J10.A28 (A21), J11.A28 (A21), J8.A28 (A21), J9.A28 (A21), RN8.11 (R10)
- net A22: now also J10.B28 (A22), J11.B28 (A22), J8.B28 (A22), J9.B28 (A22), RN9.11 (R10)
- net A23: now also J10.C28 (A23), J11.C28 (A23), J8.C28 (A23), J9.C28 (A23), RN10.11 (R10)
- net A3: now also J10.A22 (A3), J11.A22 (A3), J8.A22 (A3), J9.A22 (A3), RN8.5 (R4)
- net A4: now also J10.B22 (A4), J11.B22 (A4), J8.B22 (A4), J9.B22 (A4), RN9.5 (R4)
- net A5: now also J10.C22 (A5), J11.C22 (A5), J8.C22 (A5), J9.C22 (A5), RN10.5 (R4)
- net A6: now also J10.A23 (A6), J11.A23 (A6), J8.A23 (A6), J9.A23 (A6), RN8.6 (R5)
- net A7: now also J10.B23 (A7), J11.B23 (A7), J8.B23 (A7), J9.B23 (A7), RN9.6 (R5)
- net A8: now also J10.C23 (A8), J11.C23 (A8), J8.C23 (A8), J9.C23 (A8), RN10.6 (R5)
- net A9: now also J10.A24 (A9), J11.A24 (A9), J8.A24 (A9), J9.A24 (A9), RN8.7 (R6)
- net CLK0: now also J10.A5 (CLK0), J11.A5 (CLK0), J8.A5 (CLK0), J9.A5 (CLK0)
- net CLK1: now also J10.B5 (CLK1), J11.B5 (CLK1), J8.B5 (CLK1), J9.B5 (CLK1)
- net CS0: now also J10.C13 (CS0), J11.C13 (CS0), J8.C13 (CS0), J9.C13 (CS0), RN7.9 (R8)
- net CS1: now also J10.A14 (CS1), J11.A14 (CS1), J8.A14 (CS1), J9.A14 (CS1), RN5.10 (R9)
- net CS2: now also J10.B14 (CS2), J11.B14 (CS2), J8.B14 (CS2), J9.B14 (CS2), RN6.10 (R9)
- net CS3: now also J10.C14 (CS3), J11.C14 (CS3), J8.C14 (CS3), J9.C14 (CS3), RN7.10 (R9)
- net CTRL_1: now also J10.B7 (CTRL_1), J11.B7 (CTRL_1), J8.B7 (CTRL_1), J9.B7 (CTRL_1), RN6.3 (R2)
- net CTRL_10: now also J10.B10 (CTRL_10), J11.B10 (CTRL_10), J8.B10 (CTRL_10), J9.B10 (CTRL_10), RN6.6 (R5)
- net CTRL_11: now also J10.C10 (CTRL_11), J11.C10 (CTRL_11), J8.C10 (CTRL_11), J9.C10 (CTRL_11), RN7.6 (R5)
- net CTRL_12: now also J10.A11 (CTRL_12), J11.A11 (CTRL_12), J8.A11 (CTRL_12), J9.A11 (CTRL_12), RN5.7 (R6)
- net CTRL_13: now also J10.B11 (CTRL_13), J11.B11 (CTRL_13), J8.B11 (CTRL_13), J9.B11 (CTRL_13), RN6.7 (R6)
- net CTRL_14: now also J10.C11 (CTRL_14), J11.C11 (CTRL_14), J8.C11 (CTRL_14), J9.C11 (CTRL_14), RN7.7 (R6)
- net CTRL_15: now also J10.A12 (CTRL_15), J11.A12 (CTRL_15), J8.A12 (CTRL_15), J9.A12 (CTRL_15), RN5.8 (R7)
- net CTRL_16: now also J10.B12 (CTRL_16), J11.B12 (CTRL_16), J8.B12 (CTRL_16), J9.B12 (CTRL_16), RN6.8 (R7)
- net CTRL_17: now also J10.C12 (CTRL_17), J11.C12 (CTRL_17), J8.C12 (CTRL_17), J9.C12 (CTRL_17), RN7.8 (R7)
- net CTRL_18: now also J10.A13 (CTRL_18), J11.A13 (CTRL_18), J8.A13 (CTRL_18), J9.A13 (CTRL_18), RN5.9 (R8)
- net CTRL_19: now also J10.B13 (CTRL_19), J11.B13 (CTRL_19), J8.B13 (CTRL_19), J9.B13 (CTRL_19), RN6.9 (R8)
- net CTRL_2: now also J10.C7 (CTRL_2), J11.C7 (CTRL_2), J8.C7 (CTRL_2), J9.C7 (CTRL_2), RN7.3 (R2)
- net CTRL_3: now also J10.A8 (CTRL_3), J11.A8 (CTRL_3), J8.A8 (CTRL_3), J9.A8 (CTRL_3), RN5.4 (R3)
- net CTRL_4: now also J10.B8 (CTRL_4), J11.B8 (CTRL_4), J8.B8 (CTRL_4), J9.B8 (CTRL_4), RN6.4 (R3)
- net CTRL_5: now also J10.C8 (CTRL_5), J11.C8 (CTRL_5), J8.C8 (CTRL_5), J9.C8 (CTRL_5), RN7.4 (R3)
- net CTRL_6: now also J10.A9 (CTRL_6), J11.A9 (CTRL_6), J8.A9 (CTRL_6), J9.A9 (CTRL_6), RN5.5 (R4)
- net CTRL_7: now also J10.B9 (CTRL_7), J11.B9 (CTRL_7), J8.B9 (CTRL_7), J9.B9 (CTRL_7), RN6.5 (R4)
- net CTRL_8: now also J10.C9 (CTRL_8), J11.C9 (CTRL_8), J8.C9 (CTRL_8), J9.C9 (CTRL_8), RN7.5 (R4)
- net CTRL_9: now also J10.A10 (CTRL_9), J11.A10 (CTRL_9), J8.A10 (CTRL_9), J9.A10 (CTRL_9), RN5.6 (R5)
- net D0: now also J10.A15 (D0), J11.A15 (D0), J8.A15 (D0), J9.A15 (D0), RN5.11 (R10)
- net D1: now also J10.B15 (D1), J11.B15 (D1), J8.B15 (D1), J9.B15 (D1), RN6.11 (R10)
- net D10: now also J10.B18 (D10), J11.B18 (D10), J8.B18 (D10), J9.B18 (D10), RN6.14 (R13)
- net D11: now also J10.C18 (D11), J11.C18 (D11), J8.C18 (D11), J9.C18 (D11), RN7.14 (R13)
- net D12: now also J10.A19 (D12), J11.A19 (D12), J8.A19 (D12), J9.A19 (D12), RN8.2 (R1)
- net D13: now also J10.B19 (D13), J11.B19 (D13), J8.B19 (D13), J9.B19 (D13), RN9.2 (R1)
- net D14: now also J10.C19 (D14), J11.C19 (D14), J8.C19 (D14), J9.C19 (D14), RN10.2 (R1)
- net D15: now also J10.A20 (D15), J11.A20 (D15), J8.A20 (D15), J9.A20 (D15), RN8.3 (R2)
- net D2: now also J10.C15 (D2), J11.C15 (D2), J8.C15 (D2), J9.C15 (D2), RN7.11 (R10)
- net D3: now also J10.A16 (D3), J11.A16 (D3), J8.A16 (D3), J9.A16 (D3), RN5.12 (R11)
- net D4: now also J10.B16 (D4), J11.B16 (D4), J8.B16 (D4), J9.B16 (D4), RN6.12 (R11)
- net D5: now also J10.C16 (D5), J11.C16 (D5), J8.C16 (D5), J9.C16 (D5), RN7.12 (R11)
- net D6: now also J10.A17 (D6), J11.A17 (D6), J8.A17 (D6), J9.A17 (D6), RN5.13 (R12)
- net D7: now also J10.B17 (D7), J11.B17 (D7), J8.B17 (D7), J9.B17 (D7), RN6.13 (R12)
- net D8: now also J10.C17 (D8), J11.C17 (D8), J8.C17 (D8), J9.C17 (D8), RN7.13 (R12)
- net D9: now also J10.A18 (D9), J11.A18 (D9), J8.A18 (D9), J9.A18 (D9), RN5.14 (R13)
- net GND: now also J10.A29 (GND), J10.A32 (GND), J10.B20 (GND), J10.B29 (GND), J10.B32 (GND), J10.C20 (GND), J10.C29 (GND), J10.C3 (GND), J10.C31 (GND), J10.C32 (GND), J10.C4 (GND), J10.S1 (GND), J10.S2 (GND), J11.A29 (GND), J11.A32 (GND), J11.B20 (GND), J11.B29 (GND), J11.B32 (GND), J11.C20 (GND), J11.C29 (GND), J11.C3 (GND), J11.C31 (GND), J11.C32 (GND), J11.C4 (GND), J11.S1 (GND), J11.S2 (GND), J8.A29 (GND), J8.A32 (GND), J8.B20 (GND), J8.B29 (GND), J8.B32 (GND), J8.C20 (GND), J8.C29 (GND), J8.C3 (GND), J8.C31 (GND), J8.C32 (GND), J8.C4 (GND), J8.S1 (GND), J8.S2 (GND), J9.A29 (GND), J9.A32 (GND), J9.B20 (GND), J9.B29 (GND), J9.B32 (GND), J9.C20 (GND), J9.C29 (GND), J9.C3 (GND), J9.C31 (GND), J9.C32 (GND), J9.C4 (GND), J9.S1 (GND), J9.S2 (GND)
- net MISO: now also J10.B30 (MISO), J11.B30 (MISO), J8.B30 (MISO), J9.B30 (MISO), RN9.13 (R12)
- net MOSI: now also J10.C30 (MOSI), J11.C30 (MOSI), J8.C30 (MOSI), J9.C30 (MOSI), RN10.13 (R12)
- net SPI_CLK: now also J10.C5 (SPI_CLK), J11.C5 (SPI_CLK), J8.C5 (SPI_CLK), J9.C5 (SPI_CLK)
- net ~{PWR_OFF}: now also J10.C1 (~{PWR_OFF}), J11.C1 (~{PWR_OFF}), J8.C1 (~{PWR_OFF}), J9.C1 (~{PWR_OFF})
- net ~{RESET}: now also J10.A7 (CTRL_0), J11.A7 (CTRL_0), J8.A7 (CTRL_0), J9.A7 (CTRL_0), RN5.3 (R2)
- net ~{SHUTDOWN_RQ}: now also J10.C2 (~{SHUTDOWN_RQ}), J11.C2 (~{SHUTDOWN_RQ}), J8.C2 (~{SHUTDOWN_RQ}), J9.C2 (~{SHUTDOWN_RQ})
- net ~{SPI_INT}: now also J10.A30 (~{SPI_INT}), J11.A30 (~{SPI_INT}), J8.A30 (~{SPI_INT}), J9.A30 (~{SPI_INT}), RN8.13 (R12)
- net CART renamed ~{CART}
- net ~{CART}: now also J10.B6 (~{CART}), J11.B6 (~{CART}), J8.B6 (~{CART}), J9.B6 (~{CART}), RN6.2 (R1)
- net CLK2: no longer names the net of J6.A5 (CLK2)
- net CLK3: no longer names the net of J6.A6 (CLK3)
- net PROG renamed ~{PROG}
- net ~{PROG}: now also J10.A6 (~{PROG}), J11.A6 (~{PROG}), J8.A6 (~{PROG}), J9.A6 (~{PROG}), RN5.2 (R1)
- net SPI_CD renamed ~{SPI_CD}
- net ~{SPI_CD}: now also J10.C6 (~{SPI_CD}), J11.C6 (~{SPI_CD}), J8.C6 (~{SPI_CD}), J9.C6 (~{SPI_CD}), RN7.2 (R1)
- net SPI_CS0 renamed ~{SPI_CS0}
- net ~{SPI_CS0}: now also J10.A31 (SPI_CS0), J11.A31 (SPI_CS0), J8.A31 (SPI_CS0), J9.A31 (SPI_CS0), RN8.14 (R13)
- net SPI_CS1 renamed ~{SPI_CS1}
- net ~{SPI_CS1}: now also J10.B31 (SPI_CS1), J11.B31 (SPI_CS1), J8.B31 (SPI_CS1), J9.B31 (SPI_CS1), RN9.14 (R13)
- no-connect marks 3 -> 9
Other:
- moved on the sheet: J6C

Commit message: updated part #s
Parts:
- C10, C11, C12, C13, C14, C15, C16, C17, C8, C9: MANUFACTURER_PART_NUMBER C0603C104K3RACTU -> C1206C104K3RACTU
- J10, J11, J8, J9: MANUFACTURER_PART_NUMBER (none) -> 86093968114T55F1LF
- RN10, RN5, RN6, RN7, RN8, RN9: MANUFACTURER_PART_NUMBER (none) -> 4614X-101-472LF
