File: pBITzBackplane/Power.kicad_sch (KiCad schematic)
At the start: 20 parts, among them J1 ATX-24, Q1 BSS138, SW1 SW_Push, U1 ATtiny85-20P

Commit message: updated the pullups for the power on sequence pins
Parts:
- removed R7: 10k, Resistor_SMD:R_1206_3216Metric_Pad1.30x1.75mm_HandSolder, symbol Device:R

Commit message: updated part #s
Parts:
- C1: MANUFACTURER_PART_NUMBER C0603C104K3RACTU -> C1206C104K3RACTU
- R1, R5, R6, R8: MANUFACTURER_PART_NUMBER RC0603FR-0710KL -> RC1206FR-0710KL
- R19, R20: MANUFACTURER_PART_NUMBER RC0603FR-074K7L -> RC1206FR-074K7L
